Commit message: feat: raise camera, tilt it down, and increase resolution

File: urdf/my_robot.urdf (robot description, URDF)
Before this commit: robot my_robot, 8 links, 7 joints
Joints:
- joint camera_joint: origin xyz=0.15 0 0.04 rpy=0 0 0 -> xyz=0.15 0 0.15 rpy=0 0.35 0

Commit message: improve: camera 45deg tilt + grayscale threshold for F1 white line detection

File: urdf/my_robot.urdf (robot description, URDF)
Before this commit: robot my_robot, 8 links, 7 joints
Joints:
- joint camera_joint: origin xyz=0.15 0 0.15 rpy=0 0.35 0 -> xyz=0.18 0 0.18 rpy=0 0.785 0

Commit message: adapt: camera position from ar-tu-do reference (low 9.5cm, 21cm forward, 15deg tilt, 640x480)

File: urdf/my_robot.urdf (robot description, URDF)
Before this commit: robot my_robot, 8 links, 7 joints
Joints:
- joint camera_joint: origin xyz=0.18 0 0.18 rpy=0 0.785 0 -> xyz=0.21 0 0.095 rpy=0 0.26 0

Commit message: improve: decrease camera pitch to 5 degrees to look far ahead and anticipate curves early

File: urdf/my_robot.urdf (robot description, URDF)
Before this commit: robot my_robot, 8 links, 7 joints
Joints:
- joint camera_joint: origin xyz=0.21 0 0.095 rpy=0 0.26 0 -> xyz=0.21 0 0.095 rpy=0 0.08 0
