Commit message: feat: implement Plan B Neural Network autopilot nodes (recorder, training, and pilot) and raise camera height to 14cm

File: urdf/racer_robot.urdf (robot description, URDF)
Before this commit: robot racer_robot, 12 links, 11 joints
Joints:
- joint camera_joint: origin xyz=0.21 0 0.095 rpy=0 0.08 0 -> xyz=0.21 0 0.14 rpy=0 0.08 0
